File: ice4pi.kicad_pcb (KiCad board)
At the start: 4 copper layers, 85 x 56 mm, 32 parts, among them J1 Conn_02x03, J2 Raspberry_Pi_2_3, J3 USB_C_Receptacle_USB2.0, J4 RJ45_Amphenol_RJMG1BD3B8K1ANR, U1 ENC28J60x-SS, U2 DSC1001DE1-025.0000

Commit message: etherenet4pizero-poe-prerelease-2.0
Parts:
- added C15: 100nF 100V, Capacitor_SMD:C_0402_1005Metric, F.Cu at (106.5, 98.5)
- added D4: SMAJ58A, Diode_SMD:D_SMA, F.Cu at (104.0, 88.5)
- added LSI-U1: lsi-powermodule-7, lsi:lsi-powermodule-7, F.Cu at (96.7, 100.0)
- added R11: 5.1K, Resistor_SMD:R_0402_1005Metric, F.Cu at (59.5, 95.5)
- added R12: 0, Resistor_SMD:R_0402_1005Metric, F.Cu at (103.0, 101.2)
- added R22: 24.9K, Resistor_SMD:R_0402_1005Metric, F.Cu at (106.5, 96.0)
- added R23: 180K, Resistor_SMD:R_0402_1005Metric, F.Cu at (106.5, 92.5)
- added R24: 4.42K, Resistor_SMD:R_0402_1005Metric, F.Cu at (107.5, 92.5)
- added U3: TPS2375-1, Package_SO:TSSOP-8_4.4x3mm_P0.65mm, F.Cu at (104.0, 96.9)
- J4: value RJ45_Amphenol_RJMG1BD3B8K1ANR -> RJ45_Abracon_ARJP11A-MASA-B-A-EMU2; footprint Connector_RJ:RJ45_Amphenol_RJMG1BD3B8K1ANR -> Connector_RJ:RJ45_Abracon_ARJP11A-MA_Horizontal
- moved svg2mod 7.38 mm to (84.5, 83.6)
- moved C2 2.91 mm to (119.5, 77.5)
- moved J4 2.84 mm to (118.0, 65.0)
- moved R7 2.05 mm to (130.8, 71.5)
- moved R6 1.95 mm to (132.8, 71.5)
- moved R3 1.00 mm to (119.5, 78.5)
- moved C1 0.32 mm to (127.5, 69.5)
- moved L1 0.21 mm to (128.2, 72.8)
Connections:
- C1 pad 1: Net-(C1-Pad1) -> Net-(J4-TCT)
- C2 pad 1: Net-(C2-Pad1) -> Net-(J4-RCT)
- J3 pad A5: Net-(J3-PadA5) -> Net-(J3-CC1)
- J3 pad B5: Net-(J3-PadA5) -> Net-(J3-CC2)
- J4 pad 13: GND -> Net-(J4-Pad13)
- L1 pad 2: Net-(C1-Pad1) -> Net-(J4-TCT)
- R1 pad 1: Net-(C1-Pad1) -> Net-(J4-TCT)
- R2 pad 1: Net-(C1-Pad1) -> Net-(J4-TCT)
- R3 pad 1: Net-(C2-Pad1) -> Net-(J4-RCT)
- R4 pad 1: Net-(C2-Pad1) -> Net-(J4-RCT)
- R6 pad 1: /LEDA -> /LEDB
- R6 pad 2: Net-(R6-Pad2) -> Net-(J4-Pad13)
- R7 pad 1: /LEDB -> /LEDA
- R7 pad 2: Net-(J4-PadL1) -> Net-(J4-Pad11)
- R9 pad 1: Net-(J3-PadA5) -> Net-(J3-CC2)
Routing:
- net POE_V+: track 0.00 -> 96.7 mm, vias 0 -> 5
- net POE_V-: track 0.00 -> 69.8 mm, vias 0 -> 5
- net +5V: track 65.2 -> 95.6 mm, vias 2 -> 5
- net Net-(C2-Pad1): track 29.5 -> 0.00 mm, vias 3 -> 0
- net Net-(J4-RCT): track 0.00 -> 23.3 mm, vias 0 -> 2
- net Net-(C1-Pad1): track 23.1 -> 0.00 mm, vias 1 -> 0
- net GND: track 1.92 -> 23.3 mm, vias 9 -> 14
- net Net-(J4-PadL1): track 20.5 -> 0.00 mm
- net Net-(J4-TCT): track 0.00 -> 19.8 mm, vias 0 -> 1
- net Net-(J4-Pad13): track 0.00 -> 17.3 mm
- net Net-(LSI-U1-S2): track 0.00 -> 11.6 mm
- net /TPOUT-: track 47.0 -> 35.4 mm, vias 1 -> 3
- net Net-(J4-Pad11): track 0.00 -> 6.42 mm
- net Net-(R6-Pad2): track 6.04 -> 0.00 mm
- net /TPIN+: track 39.9 -> 34.4 mm, vias 0 -> 2
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Other:
- board text added: "ethernet4pizero-poe-1.2"
- board text removed: "ethernet4pizero-1.0"

Commit message: etherenet4pizero-poe-prerelease-2.0-1
Other:
- board text added: "ethernet4pizero-poe-2.0"
- board text removed: "ethernet4pizero-poe-1.2"
Changed lines of the file:
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@@
 		(layer "Edge.Cuts")
 	)
-	(gr_text "ethernet4pizero-poe-1.2"
+	(gr_text "ethernet4pizero-poe-2.0"
 		(at 83.75 77.5 0)
 		(layer "F.SilkS")
