File: ice4pi.kicad_sch (KiCad schematic)
At the start: 25 parts, among them J1 Conn_02x03, J2 Raspberry_Pi_2_3, J3 USB_C_Receptacle_USB2.0, J4 RJ45_Amphenol_RJMG1BD3B8K1ANR, U1 ENC28J60x-SS, U2 DSC1001DE1-025.0000

Commit message: etherenet4pizero-poe-prerelease-2.0
Parts:
- removed J4: RJ45_Amphenol_RJMG1BD3B8K1ANR, Connector_RJ:RJ45_Amphenol_RJMG1BD3B8K1ANR, symbol Connector:RJ45_Amphenol_RJMG1BD3B8K1ANR
- added C15: 100nF 100V, Capacitor_SMD:C_0402_1005Metric, symbol Device:C
- added D4: SMAJ58A, Diode_SMD:D_SMA, symbol Diode:SMAJ58A
- added J4: RJ45_Abracon_ARJP11A-MASA-B-A-EMU2, Connector_RJ:RJ45_Abracon_ARJP11A-MA_Horizontal, symbol Connector:RJ45_Abracon_ARJP11A-MASA-B-A-EMU2
- added LSI-U1: lsi-powermodule-7, lsi:lsi-powermodule-7, symbol lsi:lsi-powermodule-7
- added R11: 5.1K, Resistor_SMD:R_0402_1005Metric, symbol Device:R
- added R12: 0, Resistor_SMD:R_0402_1005Metric, symbol Device:R
- added R22: 24.9K, Resistor_SMD:R_0402_1005Metric, symbol Device:R
- added R23: 180K, Resistor_SMD:R_0402_1005Metric, symbol Device:R
- added R24: 4.42K, Resistor_SMD:R_0402_1005Metric, symbol Device:R
- added U3: TPS2375-1, Package_SO:TSSOP-8_4.4x3mm_P0.65mm, symbol Regulator_Controller:TPS2375-1
Connections:
- net +5V: now also LSI-U1.3 (VPP_OUT)
- net GND: now also J4.12, J4.14, J4.SH, LSI-U1.1 (GND), LSI-U1.4 (GND), R11.2, U3.5 (RTN)
- net LEDA: now also R7.1; no longer R6.1
- net LEDB: now also R6.1; no longer R7.1
- net TPIN+: now also J4.3 (RD+)
- net TPIN-: now also J4.6 (RD-)
- net TPOUT+: now also J4.1 (TD+)
- net TPOUT-: now also J4.2 (TD-)
- net at C1.1, L1.2, R1.1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: now also J4.4 (TCT)
- net at J3.B5 (CC2), R9.1: no longer J3.A5 (CC1)
- net at R7.2: now also J4.11
- net at R6.2: now also J4.13
- net at C2.1, R3.1, R4.1: now also J4.5 (RCT)
- new net: J3.A5 (CC1), R11.1
- new net: R22.1, U3.3 (DET)
- new net: R24.1, U3.2 (CLASS)
- new net: LSI-U1.6 (S2), R12.2
- new net: R23.1, U3.1 (ILIM)
- new net: R12.1, U3.6 (PG)
- new net POE_V+: C15.1, D4.1 (A1), J4.9 (V+), LSI-U1.2 (VPP_IN), R22.2, U3.8 (VDD)
- new net POE_V-: C15.2, D4.2 (A2), J4.10 (V-), R23.2, R24.2, U3.4 (VSS)
- no-connect marks 22 -> 32
Other:
- note removed: "2 to 1 jumper array."
- title: ethernet4pizero-1.0 -> ethernet4pizero-poe-1.0
- moved on the sheet: C5, C6, C7, C8, J1, J2, J3, R9

Commit message: etherenet4pizero-poe-prerelease-2.0-1
Other:
- title: ethernet4pizero-poe-1.0 -> ethernet4pizero-poe-2.0
Changed lines of the file:
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@@
 	(paper "A4")
 	(title_block
-		(title "ethernet4pizero-poe-1.0")
+		(title "ethernet4pizero-poe-2.0")
 		(company "Lightside Instruments AS")
 	)
@@
 	(label "TPOUT-"
 		(at 46.99 101.6 0)
-		(fields_autoplaced yes)
 		(effects
 			(font
@@
 	(label "LEDA"
 		(at 99.06 25.4 0)
-		(fields_autoplaced yes)
 		(effects
 			(font
@@
 	(label "TPOUT+"
 		(at 97.79 48.26 0)
-		(fields_autoplaced yes)
 		(effects
 			(font
@@
 	(label "CS0"
 		(at 175.26 25.4 90)
-		(fields_autoplaced yes)
 		(effects
 			(font
@@
 	(label "SI"
 		(at 57.15 30.48 0)
-		(fields_autoplaced yes)
 		(effects
 			(font
@@
 	(label "INT1"
 		(at 185.42 77.47 90)
-		(fields_autoplaced yes)
 		(effects
 			(font
@@
 	(label "LEDB"
 		(at 99.06 27.94 0)
-		(fields_autoplaced yes)
 		(effects
 			(font
@@
 	(label "TPIN+"
 		(at 48.26 104.14 0)
-		(fields_autoplaced yes)
 		(effects
 			(font
@@
 	(label "SO"
 		(at 177.8 25.4 90)
-		(fields_autoplaced yes)
 		(effects
 			(font
@@
 	(label "TPIN-"
 		(at 97.79 38.1 0)
-		(fields_autoplaced yes)
 		(effects
 			(font
@@
 	(label "CS0"
 		(at 71.12 142.24 0)
-		(fields_autoplaced yes)
 		(effects
 			(font
@@
 	(label "INT0"
 		(at 91.44 142.24 0)
-		(fields_autoplaced yes)
 		(effects
 			(font
@@
 	(label "SCK"
 		(at 57.15 35.56 0)
-		(fields_autoplaced yes)
 		(effects
 			(font
@@
 	(label "TPOUT-"
 		(at 97.79 50.8 0)
-		(fields_autoplaced yes)
 		(effects
 			(font
@@
 	(label "CLKOUT"
 		(at 36.83 66.04 0)
-		(fields_autoplaced yes)
 		(effects
 			(font
@@
 	(label "SCK"
 		(at 182.88 25.4 90)
-		(fields_autoplaced yes)
 		(effects
 			(font
@@
 	(label "INT"
 		(at 91.44 144.78 0)
-		(fields_autoplaced yes)
 		(effects
 			(font
@@
 	(label "TPIN-"
 		(at 48.26 109.22 0)
-		(fields_autoplaced yes)
 		(effects
 			(font
@@
 	(label "INT0"
 		(at 182.88 77.47 90)
-		(fields_autoplaced yes)
 		(effects
 			(font
@@
 	(label "CS"
 		(at 57.15 38.1 0)
-		(fields_autoplaced yes)
 		(effects
 			(font
@@
 	(label "LEDB"
 		(at 109.22 96.52 0)
-		(fields_autoplaced yes)
 		(effects
 			(font
@@
 	(label "CS"
 		(at 71.12 144.78 0)
-		(fields_autoplaced yes)
 		(effects
 			(font
@@
 	(label "INT1"
 		(at 91.44 147.32 0)
-		(fields_autoplaced yes)
 		(effects
 			(font
@@
 	(label "LEDA"
 		(at 109.22 106.68 0)
-		(fields_autoplaced yes)
 		(effects
 			(font
@@
 	(label "SI"
 		(at 180.34 25.4 90)
-		(fields_autoplaced yes)
 		(effects
 			(font
@@
 	(label "SO"
 		(at 57.15 33.02 0)
-		(fields_autoplaced yes)
 		(effects
 			(font
@@
 	(label "TPOUT+"
 		(at 46.99 96.52 0)
-		(fields_autoplaced yes)
 		(effects
 			(font
@@
 	(label "TPIN+"
 		(at 97.79 35.56 0)
-		(fields_autoplaced yes)
 		(effects
 			(font
@@
 	(label "INT"
 		(at 57.15 43.18 0)
-		(fields_autoplaced yes)
 		(effects
 			(font
@@
 	(label "CS1"
 		(at 71.12 147.32 0)
-		(fields_autoplaced yes)
 		(effects
 			(font
@@
 	(label "CLKOUT"
 		(at 165.1 19.05 270)
-		(fields_autoplaced yes)
 		(effects
 			(font
@@
 	(label "CS1"
 		(at 172.72 25.4 90)
-		(fields_autoplaced yes)
-		(effects
-			(font
+		(effects
+			(font

Commit message: etherenet4pizero-poe-prerelease-2.0-4
Changed lines of the file:
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@@
 (kicad_sch
-	(version 20231120)
+	(version 20250114)
 	(generator "eeschema")
-	(generator_version "8.0")
+	(generator_version "9.0")
 	(paper "A4")
 	(title_block
@@
 		(company "Lightside Instruments AS")
 	)
+	(text_box "INTERFACE"
+		(exclude_from_sim no)
+		(at 15.24 13.97 0)
+		(size 110.49 66.04)
+		(margins 0.9525 0.9525 0.9525 0.9525)
+		(stroke
+			(width 0)
+			(type default)
+		)
+		(fill
+			(type none)
+		)
+		(effects
+			(font
+				(size 1.27 1.27)
+			)
+			(justify left top)
+		)
+	)
+	(text_box "RPI"
+		(exclude_from_sim no)
+		(at 128.27 13.97 0)
+		(size 86.36 66.04)
+		(margins 0.9525 0.9525 0.9525 0.9525)
+		(stroke
+			(width 0)
+			(type default)
+		)
+		(fill
+			(type none)
+		)
+		(effects
+			(font
+				(size 1.27 1.27)
+			)
+			(justify left top)
+		)
+	)
+	(text_box "POE-2"
+		(exclude_from_sim no)
+		(at 121.92 82.55 0)
+		(size 119.38 46.99)
+		(margins 0.9525 0.9525 0.9525 0.9525)
+		(stroke
+			(width 0)
+			(type default)
+		)
+		(fill
+			(type none)
+		)
+		(effects
+			(font
+				(size 1.27 1.27)
+			)
+			(justify left top)
+		)
+	)
+	(text_box "CAPS"
+		(exclude_from_sim no)
+		(at 100.33 132.08 0)
+		(size 45.72 26.67)
+		(margins 0.9525 0.9525 0.9525 0.9525)
+		(stroke
+			(width 0)
+			(type default)
+		)
+		(fill
+			(type none)
+		)
+		(effects
+			(font
+				(size 1.27 1.27)
+			)
+			(justify left top)
+		)
+	)
+	(text_box "POE-1"
+		(exclude_from_sim no)
+		(at 15.24 82.55 0)
+		(size 104.14 46.99)
+		(margins 0.9525 0.9525 0.9525 0.9525)
+		(stroke
+			(width 0)
+			(type default)
+		)
+		(fill
+			(type none)
+		)
+		(effects
+			(font
+				(size 1.27 1.27)
+			)
+			(justify left top)
+		)
+	)
+	(text_box "USB"
+		(exclude_from_sim no)
+		(at 15.24 132.08 0)
+		(size 49.53 58.42)
+		(margins 0.9525 0.9525 0.9525 0.9525)
+		(stroke
+			(width 0)
+			(type default)
+		)
+		(fill
+			(type none)
+		)
+		(effects
+			(font
+				(size 1.27 1.27)
+			)
+			(justify left top)
+		)
+	)
+	(text_box "2 to 1 jumper array."
+		(exclude_from_sim no)
+		(at 67.31 132.08 0)
+		(size 30.48 17.78)
+		(margins 0.9525 0.9525 0.9525 0.9525)
+		(stroke
+			(width 0)
+			(type default)
+		)
+		(fill
+			(type none)
+		)
+		(effects
+			(font
+				(size 1.27 1.27)
+			)
+			(justify left top)
+		)
+	)
 	(junction
 		(at 39.37 99.06)
@@
 		)
 	)
-	(text_box "INTERFACE"
-		(exclude_from_sim no)
-		(at 15.24 13.97 0)
-		(size 110.49 66.04)
-		(stroke
-			(width 0)
-			(type default)
-		)
-		(fill
-			(type none)
-		)
-		(effects
-			(font
-				(size 1.27 1.27)
-			)
-			(justify left top)
-		)
-	)
-	(text_box "RPI"
-		(exclude_from_sim no)
-		(at 128.27 13.97 0)
-		(size 86.36 66.04)
-		(stroke
-			(width 0)
-			(type default)
-		)
-		(fill
-			(type none)
-		)
-		(effects
-			(font
-				(size 1.27 1.27)
-			)
-			(justify left top)
-		)
-	)
-	(text_box "POE-2"
-		(exclude_from_sim no)
-		(at 121.92 82.55 0)
-		(size 119.38 46.99)
-		(stroke
-			(width 0)
-			(type default)
-		)
-		(fill
-			(type none)
-		)
-		(effects
-			(font
-				(size 1.27 1.27)
-			)
-			(justify left top)
-		)
-	)
-	(text_box "CAPS"
-		(exclude_from_sim no)
-		(at 100.33 132.08 0)
-		(size 45.72 26.67)
-		(stroke
-			(width 0)
-			(type default)
-		)
-		(fill
-			(type none)
-		)
-		(effects
-			(font
-				(size 1.27 1.27)
-			)
-			(justify left top)
-		)
-	)
-	(text_box "POE-1"
-		(exclude_from_sim no)
-		(at 15.24 82.55 0)
-		(size 104.14 46.99)
-		(stroke
-			(width 0)
-			(type default)
-		)
-		(fill
-			(type none)
-		)
-		(effects
-			(font
-				(size 1.27 1.27)
-			)
-			(justify left top)
-		)
-	)
-	(text_box "USB"
-		(exclude_from_sim no)
-		(at 15.24 132.08 0)
-		(size 49.53 58.42)
-		(stroke
-			(width 0)
-			(type default)
-		)
-		(fill
-			(type none)
-		)
-		(effects
-			(font
-				(size 1.27 1.27)
-			)
-			(justify left top)
-		)
-	)
-	(text_box "2 to 1 jumper array."
-		(exclude_from_sim no)
-		(at 67.31 132.08 0)
-		(size 30.48 17.78)
-		(stroke
-			(width 0)
-			(type default)
-		)
-		(fill
-			(type none)
-		)
-		(effects
-			(font
-				(size 1.27 1.27)
-			)
-			(justify left top)
-		)
-	)
 	(label "TPOUT-"
 		(at 46.99 101.6 0)
@@
 		)
 	)
+	(embedded_fonts no)
 )
