File: ice4pi.kicad_sch (KiCad schematic)
At the start: 25 parts, among them J1 Conn_02x03, J2 Raspberry_Pi_2_3, J3 USB_C_Receptacle_USB2.0, J4 RJ45_Amphenol_RJMG1BD3B8K1ANR, U1 ENC28J60x-SS, U2 DSC1001DE1-025.0000

Commit message: Release ethernet4pizero-poe-2.0
Parts:
- removed J4: RJ45_Amphenol_RJMG1BD3B8K1ANR, Connector_RJ:RJ45_Amphenol_RJMG1BD3B8K1ANR, symbol Connector:RJ45_Amphenol_RJMG1BD3B8K1ANR
- added C15: 100nF 100V, Capacitor_SMD:C_0402_1005Metric, symbol Device:C
- added D4: SMAJ58A, Diode_SMD:D_SMA, symbol Diode:SMAJ58A
- added J4: RJ45_Abracon_ARJP11A-MASA-B-A-EMU2, Connector_RJ:RJ45_Abracon_ARJP11A-MA_Horizontal, symbol Connector:RJ45_Abracon_ARJP11A-MASA-B-A-EMU2
- added LSI-U1: lsi-powermodule-7, lsi:lsi-powermodule-7, symbol lsi:lsi-powermodule-7
- added R11: 5.1K, Resistor_SMD:R_0402_1005Metric, symbol Device:R
- added R12: 0, Resistor_SMD:R_0402_1005Metric, symbol Device:R
- added R22: 24.9K, Resistor_SMD:R_0402_1005Metric, symbol Device:R
- added R23: 180K, Resistor_SMD:R_0402_1005Metric, symbol Device:R
- added R24: 4.42K, Resistor_SMD:R_0402_1005Metric, symbol Device:R
- added U3: TPS2375-1, Package_SO:TSSOP-8_4.4x3mm_P0.65mm, symbol Regulator_Controller:TPS2375-1
Connections:
- net +5V: now also LSI-U1.3 (VPP_OUT)
- net GND: now also J4.12, J4.14, J4.SH, LSI-U1.1 (GND), LSI-U1.4 (GND), R11.2, U3.5 (RTN)
- net LEDA: now also R7.1; no longer R6.1
- net LEDB: now also R6.1; no longer R7.1
- net TPIN+: now also J4.3 (RD+)
- net TPIN-: now also J4.6 (RD-)
- net TPOUT+: now also J4.1 (TD+)
- net TPOUT-: now also J4.2 (TD-)
- net at C1.1, L1.2, R1.1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: now also J4.4 (TCT)
- net at J3.B5 (CC2), R9.1: no longer J3.A5 (CC1)
- net at R7.2: now also J4.11
- net at R6.2: now also J4.13
- net at C2.1, R3.1, R4.1: now also J4.5 (RCT)
- new net: J3.A5 (CC1), R11.1
- new net: R22.1, U3.3 (DET)
- new net: R24.1, U3.2 (CLASS)
- new net: LSI-U1.6 (S2), R12.2
- new net: R23.1, U3.1 (ILIM)
- new net: R12.1, U3.6 (PG)
- new net POE_V+: C15.1, D4.1 (A1), J4.9 (V+), LSI-U1.2 (VPP_IN), R22.2, U3.8 (VDD)
- new net POE_V-: C15.2, D4.2 (A2), J4.10 (V-), R23.2, R24.2, U3.4 (VSS)
- no-connect marks 22 -> 32
Other:
- note removed: "2 to 1 jumper array."
- title: ethernet4pizero-1.0 -> ethernet4pizero-poe-2.0
- moved on the sheet: C5, C6, C7, C8, J1, J2, J3, R9
